File: squarewavebird_sao.kicad_sch (KiCad schematic)
At the start: 14 parts, among them J1 Conn_02x03_Odd_Even

Commit message: Added teardrops, signature, C values, oriented labels, cleaned board
Parts:
- A1: now not fitted
- C1, C2, C3, C4: value C -> 0.1μF
Connections:
- no-connect marks 3 -> 4
Other:
- moved on the sheet: C1, C2, C3, C4

Commit message: Redo board for "Economic PCBA"
Parts:
- C1, C2, C3, C4: footprint Capacitor_SMD:C_0603_1608Metric -> sao:C_0603_1608Metric
Changed lines of the file:
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@@
       (effects (font (size 1.27 1.27)) (justify left))
     )
-    (property "Footprint" "Capacitor_SMD:C_0603_1608Metric" (at 141.9352 48.26 0)
+    (property "Footprint" "sao:C_0603_1608Metric" (at 141.9352 48.26 0)
       (effects (font (size 1.27 1.27)) hide)
     )
@@
       (effects (font (size 1.27 1.27)) (justify left))
     )
-    (property "Footprint" "Capacitor_SMD:C_0603_1608Metric" (at 154.6352 48.26 0)
+    (property "Footprint" "sao:C_0603_1608Metric" (at 154.6352 48.26 0)
       (effects (font (size 1.27 1.27)) hide)
     )
@@
       (effects (font (size 1.27 1.27)) (justify left))
     )
-    (property "Footprint" "Capacitor_SMD:C_0603_1608Metric" (at 129.2352 48.26 0)
+    (property "Footprint" "sao:C_0603_1608Metric" (at 129.2352 48.26 0)
       (effects (font (size 1.27 1.27)) hide)
     )
@@
       (effects (font (size 1.27 1.27)) (justify left))
     )
-    (property "Footprint" "Capacitor_SMD:C_0603_1608Metric" (at 167.3352 48.26 0)
-      (effects (font (size 1.27 1.27)) hide)
-    )
+    (property "Footprint" "sao:C_0603_1608Metric" (at 167.3352 48.26 0)
+      (effects (font (size 1.27 1.27)) hide)
+    )
